Commit message: Update mobile.xacro

File: example_description/robot/visual/mobile.xacro (robot description, xacro)
@@ -15,5 +15,4 @@
     <!-- Pure Visual (No dynamics) -->
     <xacro:macro name="manipulator_visual" params="">
-        <link name="odom"/>
         <link name="base_link">
             <origin xyz="0 0 0" rpy="0 0 0"/>
@@ -27,10 +26,4 @@
             <origin xyz="0 0 0" rpy="0 0 0"/>
         </link>
-        <!-- <link name="end_effector"/> -->
-        <joint name="base_offset" type="fixed">
-            <parent link="odom"/>
-            <child link="base_link"/>
-            <origin xyz="0 0 0" rpy="0 0 0"/>
-        </joint>
         <joint name="left_wheel" type="revolute">
             <parent link="base_link"/>

Commit message: humble

File: example_description/robot/visual/mobile.xacro (robot description, xacro)
@@ -15,4 +15,7 @@
     <!-- Pure Visual (No dynamics) -->
     <xacro:macro name="manipulator_visual" params="">
+        <link name="base_footprint">
+            <origin xyz="0 0 0" rpy="0 0 0"/>
+        </link>
         <link name="base_link">
             <origin xyz="0 0 0" rpy="0 0 0"/>
@@ -26,4 +29,18 @@
             <origin xyz="0 0 0" rpy="0 0 0"/>
         </link>
+        <link name="laser_frame">
+            <origin xyz="0 0 0" rpy="0 0 0"/>
+        </link>
+        <joint name="base_link" type="fixed">
+            <parent link="base_footprint"/>
+            <child link="base_link"/>
+            <origin xyz="0 0 0.03" rpy="0 0 0"/>
+        </joint>
+        <!-- <link name="end_effector"/> -->
+        <!-- <joint name="base_offset" type="fixed">
+            <parent link="odom"/>
+            <child link="base_link"/>
+            <origin xyz="0 0 0" rpy="0 0 0"/>
+        </joint> -->
         <joint name="left_wheel" type="revolute">
             <parent link="base_link"/>
@@ -51,5 +68,5 @@
             <parent link="base_link"/>
             <child link="imu"/>
-            <origin xyz="0 0 0" rpy="0 0 0"/>
+            <origin xyz="0 0 0.09" rpy="0 0 -1.5729"/>
         </joint>
         <joint name="steer" type="revolute">
@@ -64,4 +81,10 @@
                 effort="1000.0"/>
         </joint>
+        <joint name="laser_frame" type="fixed">
+            <parent link="imu"/>
+            <child link="laser_frame"/>
+            <origin xyz="0.255 0 0" rpy="0 0 0"/>
+            <!-- <origin xyz="0.255 0 0" rpy="3.1416 0 0"/> -->
+        </joint>
     </xacro:macro>
 </robot>
